Commit message: Updated to work with Ubuntu20 and our OxTs+VLP32C

File: launch/include/config/robot.urdf copy.xacro (robot description, xacro)
@@ -19,5 +19,5 @@
     <parent link="chassis_link" />
     <child link="velodyne" />
-    <origin xyz="-2.151 -0.224 -1.073" rpy="0 0 0" />
+    <origin xyz="2.151 0.224 1.073" rpy="0 0.26 0" />
   </joint>
   <link name="navsat_link"> </link>
