Commit message: Fixed faulty config

File: launch/include/config/robot.urdf.xacro (robot description, xacro)
@@ -19,5 +19,5 @@
     <parent link="chassis_link" />
     <child link="velodyne" />
-    <origin xyz="-2.151 -0.224 -1.073" rpy="0 0 0" />
+    <origin xyz="2.151 0.224 1.073" rpy="0 0 0" />
   </joint>
   <link name="navsat_link"> </link>

Commit message: added changed files before changeing branch

File: launch/include/config/robot.urdf.xacro (robot description, xacro)
@@ -19,5 +19,5 @@
     <parent link="chassis_link" />
     <child link="velodyne" />
-    <origin xyz="2.151 0.224 1.073" rpy="0 0 0" />
+    <origin xyz="2.026 0.033 1.059" rpy="0.0 0.20191 0.0" />
   </joint>
   <link name="navsat_link"> </link>

Commit message: Updated parameters for scan 220324

File: launch/include/config/robot.urdf.xacro (robot description, xacro)
@@ -11,17 +11,18 @@
   <link name="OxTs"> </link>
   <joint name="imu_joint" type="fixed">
-    <parent link="chassis_link" />
-    <child link="OxTs" />
+    <parent link="base_link" />
+    <child link="OxTs"/>
     <origin xyz="0 0 0" rpy="0 0 0" />
   </joint>
   <link name="velodyne"> </link>
   <joint name="velodyne_joint" type="fixed">
-    <parent link="chassis_link" />
+    <parent link="chassis_link"/>
     <child link="velodyne" />
-    <origin xyz="2.151 0.224 1.073" rpy="0 0 0" />
+    <origin xyz="0.681 0.0 0.813" rpy="-0.0 0.0 -0.0" />
+    <!-- <origin xyz="0.0 0.0 0.0" rpy="0.0 0.0 0.0" /> -->
   </joint>
   <link name="navsat_link"> </link>
   <joint name="navsat_joint" type="fixed">
-    <parent link="chassis_link" />
+    <parent link="OxTs" />
     <child link="navsat_link" />
     <origin xyz="0 0 0" rpy="0 0 0" />

Commit message: update LIO with Navsat topic instead of imu data

File: launch/include/config/robot.urdf.xacro (robot description, xacro)
@@ -19,5 +19,5 @@
     <parent link="chassis_link" />
     <child link="velodyne" />
-    <origin xyz="2.151 0.224 1.073" rpy="0 0 0" />
+    <origin xyz="0.681 0.0 0.813" rpy="0 0 0" />
   </joint>
   <link name="navsat_link"> </link>

Commit message: Added rgb to point struct

File: launch/include/config/robot.urdf.xacro (robot description, xacro)
@@ -19,5 +19,5 @@
     <parent link="chassis_link" />
     <child link="velodyne" />
-    <origin xyz="0.681 0.0 0.813" rpy="0 0 0" />
+    <origin xyz="0.681 0.0 0.813" rpy="0 0 0.03" />
   </joint>
   <link name="navsat_link"> </link>
