Commit message: migration to ROS2

File: config/robot.urdf.xacro (robot description, xacro)
@@ -9,4 +9,10 @@
     <origin xyz="0 0 0" rpy="0 0 0" />
   </joint>
+  <link name="lidar_link"> </link>
+  <joint name="lidar_joint" type="fixed">
+    <parent link="base_link" />
+    <child link="lidar_link" />
+    <origin xyz="0 0 0" rpy="0 0 0" />
+  </joint>
   <link name="imu_link"> </link>
   <joint name="imu_joint" type="fixed">
@@ -15,8 +21,8 @@
     <origin xyz="0 0 0" rpy="0 0 0" />
   </joint>
-  <link name="velodyne"> </link>
-  <joint name="velodyne_joint" type="fixed">
-    <parent link="chassis_link" />
-    <child link="velodyne" />
+  <link name="laser_sensor_frame"> </link>
+  <joint name="laser_joint" type="fixed">
+    <parent link="imu_link" />
+    <child link="laser_sensor_frame" />
     <origin xyz="0 0 0" rpy="0 0 0" />
   </joint>

Commit message: unilidar params file added and lidar and imu sync node created

File: config/robot.urdf.xacro (robot description, xacro)
@@ -13,5 +13,5 @@
     <parent link="base_link" />
     <child link="lidar_link" />
-    <origin xyz="0 0 0" rpy="0 0 0" />
+    <origin xyz="0.0 0.0 0.0" rpy="0 0 0" />
   </joint>
   <link name="imu_link"> </link>
@@ -21,9 +21,9 @@
     <origin xyz="0 0 0" rpy="0 0 0" />
   </joint>
-  <link name="laser_sensor_frame"> </link>
+  <link name="unilidar_lidar"> </link>
   <joint name="laser_joint" type="fixed">
     <parent link="imu_link" />
-    <child link="laser_sensor_frame" />
-    <origin xyz="0 0 0" rpy="0 0 0" />
+    <child link="unilidar_lidar" />
+    <origin xyz="-0.216  -0.220  0.0" rpy="0 0 0" />
   </joint>
   <link name="navsat_link"> </link>

Commit message: first commit

File: config/robot.urdf.xacro (robot description, xacro)
@@ -27,9 +27,3 @@
     <origin xyz="-0.216  -0.220  0.0" rpy="0 0 0" />
   </joint>
-  <link name="navsat_link"> </link>
-  <joint name="navsat_joint" type="fixed">
-    <parent link="chassis_link" />
-    <child link="navsat_link" />
-    <origin xyz="0 0 0" rpy="0 0 0" />
-  </joint>
 </robot>
